Commit message: Scale Lidar and Improved Resolution

File: urdf/barista_robot_model.urdf (robot description, URDF)
Before this commit: robot box_bot, 16 links, 15 joints
Links:
- link lidar: geometry visual mesh filename=package://barista_robot_description/meshes/sick_microscan3.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 scale=0.5 0.5 0.5

File: xacro/laser_scanner.xacro (robot description, xacro)
@@ -7,5 +7,5 @@
         <origin rpy="0 0 0" xyz="0 0 0" />
             <geometry>
-                <mesh filename="package://barista_robot_description/meshes/sick_microscan3.dae"/>
+                <mesh filename="package://barista_robot_description/meshes/sick_microscan3.dae" scale="0.5 0.5 0.5"/>
             </geometry>
       <material name="black"/>
@@ -23,6 +23,6 @@
           <scan>
             <horizontal>
-              <samples>200</samples>
-              <resolution>1.0</resolution>
+              <samples>720</samples>
+              <resolution>2.0</resolution>
               <min_angle>-3.14</min_angle>
               <max_angle>3.14</max_angle>
@@ -30,11 +30,11 @@
           </scan>
           <range>
-            <min>0.1</min>
-            <max>5.0</max>
+            <min>0.05</min>
+            <max>3.0</max>
           </range>
         </ray>
         <always_on>true</always_on>
         <visualize>true</visualize>
-        <update_rate>100.0</update_rate>
+        <update_rate>1</update_rate>
         <plugin name="laser" filename="libgazebo_ros_ray_sensor.so">
           <ros>
