Commit message: Added Multiple Robots - Rick and Morty

File: xacro/barista_robot_model_multiple.urdf.xacro (robot description, xacro)
@@ -6,4 +6,5 @@
 <xacro:include filename="$(find barista_robot_description)/xacro/cup_holder_tray.xacro" />
 <xacro:include filename="$(find barista_robot_description)/xacro/laser_scanner.xacro" />
+<xacro:property name="robot_name" value="$(arg robot_name)"/>
   <material name="red">
       <color rgba="1.0 0.0 0.0 1"/>
@@ -103,5 +104,5 @@
   <xacro:wheel wheel_name="left_wheel" />
   <xacro:wheel wheel_name="right_wheel" />
-  <joint name="joint_left_wheel" type="fixed">
+  <joint name="joint_left_wheel" type="continuous">
     <origin rpy="0 0 0" xyz="0 0.15 -0.0775"/>
     <child link="left_wheel"/>
@@ -111,5 +112,5 @@
     <joint_properties damping="1.0" friction="1.0"/>
   </joint>
-  <joint name="joint_right_wheel" type="fixed">
+  <joint name="joint_right_wheel" type="continuous">
     <origin rpy="0 0 0" xyz="0 -0.15 -0.0775"/>
     <child link="right_wheel"/>
@@ -209,5 +210,22 @@
     <material>Gazebo/Blue</material>
   </gazebo>
-<xacro:laser_scanner include_laser="$(arg include_laser)" />
+<xacro:laser_scanner include_laser="$(arg include_laser)" robot_name="${robot_name}" />
+<gazebo>
+    <plugin name="box_bot_joint_state" filename="libgazebo_ros_joint_state_publisher.so">
+      <ros>
+          <namespace>/${robot_name}</namespace>
+          <remapping>~/out:=joint_states</remapping>
+      </ros>
+      <update_rate>30</update_rate>
+      <joint_name>joint_left_wheel</joint_name>
+      <joint_name>joint_right_wheel</joint_name>
+      <joint_name>front_yaw_joint</joint_name>
+      <joint_name>back_yaw_joint</joint_name>
+      <joint_name>front_roll_joint</joint_name>
+      <joint_name>back_roll_joint</joint_name>
+      <joint_name>front_pitch_joint</joint_name>
+      <joint_name>back_pitch_joint</joint_name>
+    </plugin>
+  </gazebo>
   <!-- Differential drive -->
   <gazebo>
@@ -225,6 +243,10 @@
       <publish_odom>true</publish_odom>
       <publish_odom_tf>true</publish_odom_tf>
-      <odometry_frame>odom</odometry_frame>
-      <robot_base_frame>base_link</robot_base_frame>
+      <odometry_frame>${robot_name}/odom</odometry_frame>
+      <robot_base_frame>${robot_name}/base_link</robot_base_frame>
+        <ros>
+            <namespace>/${robot_name}</namespace>
+            <remapping>~/out:=cmd_vel</remapping>
+        </ros>
     </plugin>
   </gazebo>

Commit message: Fixed LIDAR point issue in RViz

File: xacro/barista_robot_model_multiple.urdf.xacro (robot description, xacro)
@@ -7,7 +7,11 @@
 <xacro:include filename="$(find barista_robot_description)/xacro/laser_scanner.xacro" />
 <xacro:property name="robot_name" value="$(arg robot_name)"/>
+<xacro:property name="gazebo_color" value="$(arg gazebo_color)" />
   <material name="red">
       <color rgba="1.0 0.0 0.0 1"/>
   </material>
+  <material name="rick_color">
+      <color rgba="1.0 0.0 0.0 1"/>
+  </material>
   <material name="green_light">
       <color rgba="0.0 1.0 0.0 1"/>
@@ -19,4 +23,7 @@
       <color rgba="0.0 0.0 1.0 1"/>
   </material>
+    <material name="morty_color">
+      <color rgba="0.0 0.0 1.0 1"/>
+  </material>
   <material name="black">
       <color rgba="0.0 0.0 0.0 1"/>
@@ -30,4 +37,5 @@
   <link name="base_link">
   </link>
+<material name="rick" script="model://barista_robot_description/materials/rick.material"/>
   <!-- Body -->
   <link name="chassis">
@@ -36,5 +44,5 @@
         <cylinder length="0.155" radius="0.178"/>
       </geometry>
-      <material name="red"/>
+        <material name="${robot_name}_color"/>
     </visual>
     <collision>
@@ -54,6 +62,6 @@
     <child link="chassis" />
   </joint>
-    <gazebo reference="chassis">
-        <material>Gazebo/Red</material>
+  <gazebo reference="chassis">
+    <material>${gazebo_color}</material>
   </gazebo>
   <xacro:standoff rod_name="rod_1" />
@@ -100,5 +108,5 @@
 </joint>
 <gazebo reference="cupholder_link">
-    <material>Gazebo/Red</material>
+    <material>${gazebo_color}</material>
 </gazebo>
   <xacro:wheel wheel_name="left_wheel" />
@@ -212,5 +220,5 @@
   <xacro:laser_scanner include_laser="$(arg include_laser)" robot_name="${robot_name}" />
     <gazebo>
-    <plugin name="box_bot_joint_state" filename="libgazebo_ros_joint_state_publisher.so">
+    <plugin name="joint_state" filename="libgazebo_ros_joint_state_publisher.so">
       <ros>
           <namespace>/${robot_name}</namespace>

File: xacro/laser_scanner.xacro (robot description, xacro)
@@ -32,5 +32,5 @@
             </scan>
             <range>
-              <min>0.025</min>
+              <min>0.1</min>
               <max>5.0</max>
             </range>
@@ -40,6 +40,8 @@
           <update_rate>50.0</update_rate>
           <plugin name="laser" filename="libgazebo_ros_ray_sensor.so">
+            <frame_name>${robot_name}/base_link</frame_name>
+            <topic_name>${robot_name}/scan</topic_name>
             <ros>
-                <namespace>${robot_name}</namespace>
+              <namespace>${robot_name}</namespace>
               <remapping>~/out:=scan</remapping>
             </ros>
